File: Mutsu.kicad_pcb (KiCad board)
At the start: 2 copper layers, 302 x 92.5 mm, 135 parts, among them SW1 SW_SPST, SW10 SW_SPST, SW11 SW_SPST, SW12 SW_SPST, SW13 SW_SPST, SW14 SW_SPST, SW15 SW_SPST, SW16 SW_SPST, SW17 SW_SPST, SW18 SW_SPST, SW19 SW_SPST, SW2 SW_SPST, SW20 SW_SPST, SW21 SW_SPST, SW22 SW_SPST, SW23 SW_SPST, SW24 SW_SPST, SW25 SW_SPST, SW26 SW_SPST, SW27 SW_SPST, SW28 SW_SPST, SW29 SW_SPST, SW3 SW_SPST, SW30 SW_SPST, SW31 SW_SPST, SW32 SW_SPST, SW33 SW_SPST, SW34 SW_SPST, SW35 SW_SPST, SW36 SW_SPST, SW37 SW_SPST, SW38 SW_SPST, SW39 SW_SPST, SW4 SW_SPST, SW40 SW_SPST, SW41 SW_SPST, SW42 SW_SPST, SW43 SW_SPST, SW44 SW_SPST, SW45 SW_SPST, SW46 SW_SPST, SW47 SW_SPST, SW48 SW_SPST, SW49 SW_SPST, SW5 SW_SPST, SW50 SW_SPST, SW51 SW_SPST, SW52 SW_SPST, SW53 SW_SPST, SW54 SW_SPST, SW55 SW_SPST, SW56 SW_SPST, SW57 SW_SPST, SW58 SW_SPST, SW59 SW_SPST, SW6 SW_SPST, SW60 SW_SPST, SW61 SW_SPST, SW62 SW_SPST, SW63 SW_SPST, SW64 SW_SPST, SW65 SW_SPST, SW66 SW_SPST, SW67 SW_SPST, SW7 SW_SPST, SW8 SW_SPST, SW9 SW_SPST, U1 RP2350A-QFN60

Commit message: fourth commit
Other:
- board text added: "^ microcontroller"
- board text added: "spacebar --->"
Changed lines of the file:
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@@
 			(layer "F.Mask"
 				(type "Top Solder Mask")
-				(color "Black")
+				(color "Purple")
 				(thickness 0.01)
 			)
@@
 			(layer "B.Mask"
 				(type "Bottom Solder Mask")
-				(color "Black")
+				(color "Purple")
 				(thickness 0.01)
 			)
@@
 			(at 0 -5.55 0)
 			(layer "F.SilkS")
+			(hide yes)
 			(effects
 				(font
@@
 		)
 	)
+	(gr_text "    ^\nmicrocontroller\n"
+		(at 304.5 47 0)
+		(layer "F.SilkS")
+		(effects
+			(font
+				(size 1 1)
+				(thickness 0.25)
+				(bold yes)
+			)
+			(justify left bottom)
+		)
+	)
 	(gr_text ":)"
 		(at 276 73.5 90)
@@
 		)
 	)
+	(gr_text "spacebar --->"
+		(at 125 114.5 0)
+		(layer "F.SilkS")
+		(effects
+			(font
+				(size 2 2)
+				(thickness 0.5)
+				(bold yes)
+			)
+			(justify left bottom)
+		)
+	)
 	(gr_text ":)"
 		(at 110 90.5 0)
@@
 		)
 		(gr_text "92.5"
-			(at 30.9 76.25 90)
+			(at 30.8 76.25 90)
 			(layer "F.SilkS")
 			(effects
 				(font
 					(size 1 1)
-					(thickness 0.1)
+					(thickness 0.2)
+					(bold yes)
 				)
 			)

Commit message: hehe
Parts:
- added C10: 1u, Capacitor_SMD:C_0402_1005Metric, F.Cu at (213.5, 140.0)
- added C11: 100n, Capacitor_SMD:C_0402_1005Metric, F.Cu at (172.5, 143.5)
- added C12: 100n, Capacitor_SMD:C_0402_1005Metric, F.Cu at (172.5, 145.5)
- added C13: 100n, Capacitor_SMD:C_0402_1005Metric, F.Cu at (172.5, 147.5)
- added C14: 100n, Capacitor_SMD:C_0402_1005Metric, F.Cu at (172.5, 149.4)
- added C15: 100n, Capacitor_SMD:C_0402_1005Metric, F.Cu at (172.5, 151.4)
- added C18: 100n, Capacitor_SMD:C_0402_1005Metric, F.Cu at (172.5, 153.4)
- added C5: 100n, Capacitor_SMD:C_0402_1005Metric, F.Cu at (213.5, 132.1)
- added C6: 100n, Capacitor_SMD:C_0402_1005Metric, F.Cu at (213.5, 134.1)
- added C7: 100n, Capacitor_SMD:C_0402_1005Metric, F.Cu at (213.5, 136.0)
- added C8: 1u, Capacitor_SMD:C_0402_1005Metric, F.Cu at (213.5, 138.0)
- added C9: 100n, Capacitor_SMD:C_0402_1005Metric, F.Cu at (172.5, 141.6)
- added C9: 100n, Capacitor_SMD:C_0402_1005Metric, F.Cu at (172.5, 139.6)
- added J1: USB_C_Receptacle_USB2.0_16P, Connector_USB:USB_C_Receptacle_GCT_USB4105-xx-A_16P_TopMnt_Horizontal, B.Cu at (280.9, 32.2)
- added J2: Conn_01x02, Connector_PinHeader_2.54mm:PinHeader_1x02_P2.54mm_Vertical, F.Cu at (209.8, 133.4)
- added R1: 5.1k, Resistor_SMD:R_0402_1005Metric, B.Cu at (284.5, 38.5)
- added R3: 1k, Resistor_SMD:R_0402_1005Metric, F.Cu at (208.9, 139.2)
- added R4: DNF, Resistor_SMD:R_0402_1005Metric, F.Cu at (208.9, 141.2)
- added R5: 33, Resistor_SMD:R_0402_1005Metric, F.Cu at (175.4, 139.6)
- added U4: AP2205-33Y-13, Package_TO_SOT_SMD:SOT-89-3, B.Cu at (277.5, 41.5)
- U1: moved to B.Cu
- moved U1 1.11 mm to (308.7, 39.5), turned to 135 degrees
Connections:
- U1 pad 1: unconnected-(U1-IOVDD-Pad1) -> +3V3
- U1 pad 11: unconnected-(U1-IOVDD-Pad11) -> +3V3
- U1 pad 2: column14 -> column15
- U1 pad 20: unconnected-(U1-IOVDD-Pad20) -> +3V3
- U1 pad 29: column15 -> column14
- U1 pad 30: unconnected-(U1-IOVDD-Pad30) -> +3V3
- U1 pad 38: unconnected-(U1-IOVDD-Pad38) -> +3V3
- U1 pad 44: unconnected-(U1-ADC_AVDD-Pad44) -> +3V3
- U1 pad 45: unconnected-(U1-IOVDD-Pad45) -> +3V3
- U1 pad 46: unconnected-(U1-VREG_AVDD-Pad46) -> /VREG_AVDD
- U1 pad 47: unconnected-(U1-VREG_PGND-Pad47) -> GND
- U1 pad 48: unconnected-(U1-VREG_LX-Pad48) -> /VREG_LX
- U1 pad 49: unconnected-(U1-VREG_VIN-Pad49) -> +3V3
- U1 pad 50: unconnected-(U1-VREG_FB-Pad50) -> +1V1
- U1 pad 51: unconnected-(U1-USB_DM-Pad51) -> D-
- U1 pad 52: unconnected-(U1-USB_DP-Pad52) -> D+
- U1 pad 53: unconnected-(U1-USB_OTP_VDD-Pad53) -> +3V3
- U1 pad 54: unconnected-(U1-QSPI_IOVDD-Pad54) -> +3V3
- U1 pad 61: unconnected-(U1-GND-Pad61) -> GND
Routing:
- net column1: track 357.8 -> 85.1 mm
- net column2: track 347.3 -> 94.5 mm
- net column3: track 324.2 -> 91.0 mm
- net column4: track 281.0 -> 67.0 mm
- net column5: track 261.8 -> 67.0 mm
- net column6: track 262.6 -> 87.0 mm
- net column7: track 223.5 -> 67.0 mm
- net column8: track 204.4 -> 67.2 mm
- net column9: track 185.1 -> 67.0 mm
- net column10: track 185.9 -> 87.0 mm
- net row5: track 390.6 -> 296.1 mm
- net column11: track 166.8 -> 87.0 mm
- net row4: track 369.7 -> 294.4 mm
- net column12: track 155.0 -> 94.4 mm
- net row3: track 358.0 -> 299.9 mm
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Other:
- board size 302 x 92.5 mm -> 307 x 95.5 mm
- board text added: "307"
- board text added: "92.5"
