File: Mutsu.kicad_sch (KiCad schematic)
At the start: 135 parts, among them SW1 SW_SPST, SW10 SW_SPST, SW11 SW_SPST, SW12 SW_SPST, SW13 SW_SPST, SW14 SW_SPST, SW15 SW_SPST, SW16 SW_SPST, SW17 SW_SPST, SW18 SW_SPST, SW19 SW_SPST, SW2 SW_SPST, SW20 SW_SPST, SW21 SW_SPST, SW22 SW_SPST, SW23 SW_SPST, SW24 SW_SPST, SW25 SW_SPST, SW26 SW_SPST, SW27 SW_SPST, SW28 SW_SPST, SW29 SW_SPST, SW3 SW_SPST, SW30 SW_SPST, SW31 SW_SPST, SW32 SW_SPST, SW33 SW_SPST, SW34 SW_SPST, SW35 SW_SPST, SW36 SW_SPST, SW37 SW_SPST, SW38 SW_SPST, SW39 SW_SPST, SW4 SW_SPST, SW40 SW_SPST, SW41 SW_SPST, SW42 SW_SPST, SW43 SW_SPST, SW44 SW_SPST, SW45 SW_SPST, SW46 SW_SPST, SW47 SW_SPST, SW48 SW_SPST, SW49 SW_SPST, SW5 SW_SPST, SW50 SW_SPST, SW51 SW_SPST, SW52 SW_SPST, SW53 SW_SPST, SW54 SW_SPST, SW55 SW_SPST, SW56 SW_SPST, SW57 SW_SPST, SW58 SW_SPST, SW59 SW_SPST, SW6 SW_SPST, SW60 SW_SPST, SW61 SW_SPST, SW62 SW_SPST, SW63 SW_SPST, SW64 SW_SPST, SW65 SW_SPST, SW66 SW_SPST, SW67 SW_SPST, SW7 SW_SPST, SW8 SW_SPST, SW9 SW_SPST, U1 RP2350A-QFN60

Commit message: hehe
Parts:
- removed U1: RP2350A-QFN60, extra footprints:RP2350A_QFN-60_EP_7.75x7.75_Pitch0.4mm, symbol rp2350b-qfn60:RP2350A-QFN60
- added C1, C2, C3: C_Small, symbol Device:C_Small
- added C10, C8: 1u, Capacitor_SMD:C_0402_1005Metric, symbol Device:C
- added C11, C12, C13, C14, C15, C5, C6, C7, C9: 100n, Capacitor_SMD:C_0402_1005Metric, symbol Device:C
- added J1: USB_C_Receptacle_USB2.0_16P, Connector_USB:USB_C_Receptacle_GCT_USB4105-xx-A_16P_TopMnt_Horizontal, symbol Connector:USB_C_Receptacle_USB2.0_16P
- added J2: Conn_01x02, Connector_PinHeader_2.54mm:PinHeader_1x02_P2.54mm_Vertical, symbol Connector_Generic:Conn_01x02
- added R1, R2: 5.1k, symbol Device:R
- added R3: 1k, Resistor_SMD:R_0402_1005Metric, symbol Device:R
- added R4: DNF, Resistor_SMD:R_0402_1005Metric, symbol Device:R
- added TP1, TP2: TestPoint, symbol Connector:TestPoint
- added U2: W25Q128JVS, Package_SO:SOIC-8_5.23x5.23mm_P1.27mm, symbol Memory_Flash:W25Q128JVS
- added U3: RP2040, RP2040_minimal:RP2040-QFN-56, symbol MCU_RaspberryPi_RP2040:RP2040
- added U4: AP2205-33Y-13, Package_TO_SOT_SMD:SOT-89-3, symbol Regulator_Linear:AP2204R-3.3
Connections:
- net column1: now also U3.30 (GPIO19)
- net column10: now also U3.13 (GPIO10)
- net column11: now also U3.12 (GPIO9)
- net column12: now also U3.11 (GPIO8)
- net column13: now also U3.9 (GPIO7)
- net column14: now also U3.8 (GPIO6)
- net column15: now also U3.7 (GPIO5)
- net column2: now also U3.29 (GPIO18)
- net column3: now also U3.28 (GPIO17)
- net column4: now also U3.27 (GPIO16)
- net column5: now also U3.18 (GPIO15)
- net column6: now also U3.17 (GPIO14)
- net column7: now also U3.16 (GPIO13)
- net column8: now also U3.15 (GPIO12)
- net column9: now also U3.14 (GPIO11)
- net row1: now also U3.6 (GPIO4)
- net row2: now also U3.5 (GPIO3)
- net row3: now also U3.4 (GPIO2)
- net row4: now also U3.3 (GPIO1)
- net row5: now also U3.2 (GPIO0)
- new net: C11.2, C12.2, C13.2, C14.2, C15.2, C9.2
- new net: J1.A5 (CC1), R1.1
- new net: J1.B5 (CC2), R2.1
- new net +1V1: C6.1, C7.1, C8.1, U3.23 (DVDD), U3.45 (VREG_VOUT), U3.50 (DVDD)
- new net +3V3: C1.1, C10.1, C11.1, C12.1, C13.1, C14.1, C15.1, C2.2, C5.1, C9.1, R4.1, U2.8 (VCC), U3.1 (IOVDD), U3.10 (IOVDD), U3.22 (IOVDD), U3.33 (IOVDD), U3.42 (IOVDD), U3.43 (ADC_AVDD), U3.44 (VREG_IN), U3.48 (USB_VDD), U3.49 (IOVDD), U4.3 (VOUT)
- new net +5V: C3.1, J1.A4 (VBUS), J1.A9 (VBUS), J1.B4 (VBUS), J1.B9 (VBUS), TP1.1, U4.1 (VIN)
- new net D+: J1.A7 (D-), J1.B7 (D-), U3.47 (USB_DP)
- new net D-: J1.A6 (D+), J1.B6 (D+), U3.46 (USB_DM)
- new net GND: C1.2, C10.2, C2.1, C3.2, C5.2, C6.2, C7.2, C8.2, J1.A1 (GND), J1.A12 (GND), J1.B1 (GND), J1.B12 (GND), J2.2 (Pin_2), R1.2, R2.2, U2.4 (GND), U3.19 (TESTEN), U3.57 (GND), U4.2 (GND)
- new net QSPI_SCLK: U2.6 (CLK), U3.52 (QSPI_SCLK)
- new net QSPI_SD0: U2.5 (DI(IO0)), U3.53 (QSPI_SD0)
- new net QSPI_SD1: U2.2 (DO(IO1)), U3.55 (QSPI_SD1)
- new net QSPI_SD2: U2.3 (IO2), U3.54 (QSPI_SD2)
- new net QSPI_SD3: U2.7 (IO3), U3.51 (QSPI_SD3)
- new net QSPI_SS: R3.1, R4.2, U2.1 (~{CS}), U3.56 (QSPI_SS)
- new net ~{USB_BOOT}: J2.1 (Pin_1), R3.2
- no-connect marks 0 -> 3
Other:
- note added: "Flash"
- note added: "Make sure C10 is close to pin 44 of RP2040"
